File: ISOVan.kicad_pcb (KiCad board)
At the start: 2 copper layers, 100 parts, among them SW1 SW_Push, U1 ATmega32U4-AU, Y1 16MHz

Commit message: place components
Parts:
- C7: footprint Diode_SMD:D_SOD-123 -> Capacitor_SMD:C_0805_2012Metric
- moved D43 240.2 mm to (208.4, 216.7), turned to 90 degrees
- moved D36 234.5 mm to (170.3, 216.7), turned to 90 degrees
- moved D40 231.8 mm to (189.3, 216.7), turned to 90 degrees
- moved D39 228.7 mm to (175.0, 197.6), turned to 90 degrees
- moved D19 227.4 mm to (89.3, 178.6), turned to 90 degrees
- moved D42 226.1 mm to (201.2, 197.6), turned to 90 degrees
- moved D38 221.5 mm to (184.5, 178.6), turned to 90 degrees
- moved D41 219.5 mm to (206.0, 169.1), turned to 90 degrees
- moved D35 217.7 mm to (156.0, 197.6), turned to 90 degrees
- moved D2 217.5 mm to (-15.5, 197.6), turned to 90 degrees
- moved C5 214.9 mm to (89.3, 225.0), turned to 180 degrees
- moved D37 214.7 mm to (179.8, 159.5), turned to 90 degrees
- moved D3 210.2 mm to (-11.9, 216.7), turned to 90 degrees
- moved D34 209.1 mm to (165.5, 178.6), turned to 90 degrees
- moved R3 206.0 mm to (77.4, 213.1), turned to 90 degrees
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
Commit message: place screw holes
Parts:
- added REF**: MountingHole_2.2mm_M2_Pad, MountingHole:MountingHole_2.2mm_M2_Pad, F.Cu at (108.3, 19.8)
- added REF**: MountingHole_2.2mm_M2_Pad, MountingHole:MountingHole_2.2mm_M2_Pad, F.Cu at (183.2, 66.3)
- added REF**: MountingHole_2.2mm_M2_Pad, MountingHole:MountingHole_2.2mm_M2_Pad, F.Cu at (77.5, 66.1)
- added REF**: MountingHole_2.2mm_M2_Pad, MountingHole:MountingHole_2.2mm_M2_Pad, F.Cu at (30.6, 54.6)
- added REF**: MountingHole_2.2mm_M2_Pad, MountingHole:MountingHole_2.2mm_M2_Pad, F.Cu at (138.9, 38.9)
- added REF**: MountingHole_2.2mm_M2_Pad, MountingHole:MountingHole_2.2mm_M2_Pad, F.Cu at (211.5, 17.5)
- added REF**: MountingHole_2.2mm_M2_Pad, MountingHole:MountingHole_2.2mm_M2_Pad, F.Cu at (32.1, 19.8)
- moved R1 268.7 mm to (218.1, 18.6)
- moved R2 268.7 mm to (215.2, 18.6)
- moved C1 153.1 mm to (129.5, 63.9)
- moved C2 153.1 mm to (117.6, 59.1)
- moved C3 153.1 mm to (123.5, 55.5)
- moved C4 153.1 mm to (114.0, 55.5)
- moved C6 153.1 mm to (116.4, 75.8)
- moved C7 153.1 mm to (110.5, 69.8)
- moved D1 153.1 mm to (3.29, 19.8)
- moved D10 153.1 mm to (59.3, 48.4)
- moved D11 153.1 mm to (68.8, 67.4)
- moved D13 153.1 mm to (85.4, 29.3)
- moved D14 153.1 mm to (75.9, 48.4)
- moved D16 153.1 mm to (104.5, 29.3)
- moved D17 153.1 mm to (95.0, 48.4)
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Other:
- board outline added: 244.5 x 77.8 mm

Commit message: new layout
Parts:
- removed REF** (x7): MountingHole_2.2mm_M2_Pad, MountingHole:MountingHole_2.2mm_M2_Pad
- MX11, MX3: footprint MX_Only:MXOnly-1.25U-NoLED -> MX_Only:MXOnly-1U-NoLED
- MX2: footprint MX_Only:MXOnly-1U-NoLED -> MX_Only:MXOnly-1.75U-NoLED
- MX31: renamed from MX32; value Left -> /; footprint MX_Only:MXOnly-1U-NoLED -> MX_Only:MXOnly-1.5U-NoLED
- MX36: value Down -> Left
- MX39: renamed from MX6; value \ -> Up
- MX40: value Up -> Down
- MX42: footprint MX_Only:MXOnly-1.75U-NoLED -> MX_Only:MXOnly-1U-NoLED
- moved D39 188.2 mm to (226.1, 48.4)
- moved MX39 185.6 mm to (215.1, 48.5)
- moved MX15 9.65 mm to (88.9, 67.5)
- moved MX25 9.65 mm to (136.5, 67.5)
- moved D42 7.27 mm to (242.7, 48.4)
- moved MX11 7.27 mm to (53.2, 67.5)
- moved MX2 7.02 mm to (17.5, 48.5)
- moved MX42 7.02 mm to (234.2, 48.5)
- moved MX10 4.88 mm to (62.7, 48.5)
- moved MX14 4.88 mm to (81.8, 48.5)
- moved MX18 4.88 mm to (100.8, 48.5)
- moved MX24 4.88 mm to (138.9, 48.5)
- moved MX28 4.88 mm to (158.0, 48.5)
- moved MX31 4.88 mm to (172.2, 67.5)
- moved MX35 4.88 mm to (196.1, 48.5)
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- renumbered D14 to D10, D17 to D14, D21 to D15, D15 to D16, D16 to D17, D20 to D18, D18 to D19, D19 to D20, D24 to D21, D27 to D24, D28 to D25, D25 to D26, D26 to D27, D31 to D28, D32 to D31, D35 to D32, D39 to D35, D6 to D39, D10 to D6, MX14 to MX10, MX17 to MX14, MX21 to MX15, MX15 to MX16, MX16 to MX17, MX20 to MX18, MX18 to MX19, MX19 to MX20, MX24 to MX21, MX27 to MX24, MX28 to MX25, MX25 to MX26, MX26 to MX27, MX31 to MX28, MX35 to MX32, MX39 to MX35, MX10 to MX6
Connections:
- MX10 pad 1: Col3 -> Net-(MX10-Pad1)
- MX11 pad 1: Col2 -> Net-(MX10-Pad1)
- MX14 pad 1: Col4 -> Net-(MX14-Pad1)
- MX15 pad 1: Col5 -> Net-(MX14-Pad1)
- MX18 pad 1: Col5 -> (no net)
- MX21 pad 1: Col6 -> Col5
- MX24 pad 1: Col7 -> Net-(MX24-Pad1)
- MX25 pad 1: Col7 -> Net-(MX24-Pad1)
- MX28 pad 1: Col8 -> Col7
- MX31 pad 1: Col8 -> (no net)
- MX32 pad 1: Col9 -> (no net)
- MX35 pad 1: Col10 -> Col9
- MX39 pad 1: Col1 -> Col10
- MX6 pad 1: Col2 -> Col1

Commit message: Route matrix and change layout again
Parts:
- added REF**: MountingHole_2.2mm_M2_Pad, MountingHole:MountingHole_2.2mm_M2_Pad, F.Cu at (183.2, 66.3)
- added REF**: MountingHole_2.2mm_M2_Pad, MountingHole:MountingHole_2.2mm_M2_Pad, F.Cu at (77.5, 66.1)
- added REF**: MountingHole_2.2mm_M2_Pad, MountingHole:MountingHole_2.2mm_M2_Pad, F.Cu at (30.6, 54.6)
- added REF**: MountingHole_2.2mm_M2_Pad, MountingHole:MountingHole_2.2mm_M2_Pad, F.Cu at (211.5, 17.5)
- added REF**: MountingHole_2.2mm_M2_Pad, MountingHole:MountingHole_2.2mm_M2_Pad, F.Cu at (108.3, 19.8)
- added REF**: MountingHole_2.2mm_M2_Pad, MountingHole:MountingHole_2.2mm_M2_Pad, F.Cu at (32.1, 19.8)
- MX11: footprint MX_Only:MXOnly-1U-NoLED -> MX_Only:MXOnly-1.25U-NoLED
- MX15: footprint MX_Only:MXOnly-2.75U-ReversedStabilizers-NoLED -> MX_Only:MXOnly-2.25U-ReversedStabilizers-NoLED
- MX25: footprint MX_Only:MXOnly-2.25U-ReversedStabilizers-NoLED -> MX_Only:MXOnly-2U-FLIPPED-ReversedStabilizers
- MX3: footprint MX_Only:MXOnly-1U-NoLED -> MX_Only:MXOnly-1.5U-NoLED
- moved D18 21.2 mm to (92.8, 48.1)
- moved D11 14.7 mm to (55.2, 73.0)
- moved D31 12.0 mm to (175.6, 74.3)
- moved MX11 11.9 mm to (65.1, 67.5)
- moved MX15 9.52 mm to (98.4, 67.5)
- moved MX7 9.51 mm to (41.3, 67.5)
- moved SW1 7.64 mm to (231.6, 37.2)
- moved D6 7.34 mm to (52.0, 47.7)
- moved D2 7.28 mm to (26.1, 48.4)
- moved D15 6.26 mm to (104.1, 73.0)
- moved D10 5.04 mm to (71.0, 47.6)
- moved D24 4.97 mm to (147.2, 48.3)
- moved D21 4.92 mm to (128.2, 48.3)
- moved D14 4.83 mm to (90.2, 48.1)
- moved D28 4.82 mm to (166.3, 48.3)
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Connections:
- MX10 pad 1: Net-(MX10-Pad1) -> Col2
- MX11 pad 1: Net-(MX10-Pad1) -> Col2
- MX14 pad 1: Net-(MX14-Pad1) -> Col3
- MX15 pad 1: Net-(MX14-Pad1) -> Col4
- MX18 pad 1: (no net) -> Col4
- MX24 pad 1: Net-(MX24-Pad1) -> Col6
- MX25 pad 1: Net-(MX24-Pad1) -> Col6
- MX31 pad 1: (no net) -> Col8
- MX32 pad 1: (no net) -> Col8
Routing:
- net Row3: track 0.00 -> 308.5 mm
- net Row2: track 0.00 -> 307.0 mm, vias 0 -> 4
- net Row0: track 0.00 -> 306.8 mm
- net Row1: track 0.00 -> 229.6 mm
- net Col8: track 0.00 -> 64.4 mm
- net Col6: track 0.00 -> 63.2 mm
- net Col1: track 0.00 -> 62.6 mm
- net Col9: track 0.00 -> 62.4 mm
- net Col2: track 0.00 -> 62.2 mm
- net Col4: track 0.00 -> 62.1 mm
- net Col10: track 0.00 -> 62.0 mm
- net Col11: track 0.00 -> 49.1 mm
- net GND: track 0.00 -> 47.4 mm
- net Col5: track 0.00 -> 43.1 mm
- net Col7: track 0.00 -> 42.0 mm
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