File: ISOVan.sch (KiCad schematic (older format))
At the start: 14 parts

Commit message: start matrix
Parts:
- added D? (x22): SOD-123, symbol Device:D_Small
- added MX?: Esc, symbol MX_Alps_Hybrid:MX-NoLED
- added MX?: Q, symbol MX_Alps_Hybrid:MX-NoLED
- added MX?: W, symbol MX_Alps_Hybrid:MX-NoLED
- added MX?: E, symbol MX_Alps_Hybrid:MX-NoLED
- added MX?: R, symbol MX_Alps_Hybrid:MX-NoLED
- added MX?: T, symbol MX_Alps_Hybrid:MX-NoLED
- added MX?: Y, symbol MX_Alps_Hybrid:MX-NoLED
- added MX?: U, symbol MX_Alps_Hybrid:MX-NoLED
- added MX?: I, symbol MX_Alps_Hybrid:MX-NoLED
- added MX?: O, symbol MX_Alps_Hybrid:MX-NoLED
- added MX?: P, symbol MX_Alps_Hybrid:MX-NoLED
- added MX?: Ent, symbol MX_Alps_Hybrid:MX-NoLED
- added MX?: ;, symbol MX_Alps_Hybrid:MX-NoLED
- added MX?: L, symbol MX_Alps_Hybrid:MX-NoLED
- added MX?: K, symbol MX_Alps_Hybrid:MX-NoLED
- added MX?: J, symbol MX_Alps_Hybrid:MX-NoLED
- added MX?: H, symbol MX_Alps_Hybrid:MX-NoLED
- added MX?: G, symbol MX_Alps_Hybrid:MX-NoLED
- added MX?: F, symbol MX_Alps_Hybrid:MX-NoLED
- added MX?: D, symbol MX_Alps_Hybrid:MX-NoLED
- added MX?: S, symbol MX_Alps_Hybrid:MX-NoLED
- added MX?: A, symbol MX_Alps_Hybrid:MX-NoLED
Connections:
- new net: D?.2 (A), MX?.2 (ROW) (x22)
- new net Col0: MX?.1 (COL)
- new net Col1: MX?.1 (COL), MX?.1 (COL)
- new net Col10: MX?.1 (COL), MX?.1 (COL)
- new net Col11: MX?.1 (COL)
- new net Col2: MX?.1 (COL), MX?.1 (COL)
- new net Col3: MX?.1 (COL), MX?.1 (COL)
- new net Col4: MX?.1 (COL), MX?.1 (COL)
- new net Col5: MX?.1 (COL), MX?.1 (COL)
- new net Col6: MX?.1 (COL), MX?.1 (COL)
- new net Col7: MX?.1 (COL), MX?.1 (COL)
- new net Col8: MX?.1 (COL), MX?.1 (COL)
- new net Col9: MX?.1 (COL), MX?.1 (COL)
- new net Row0: D?.1 (K), D?.1 (K), D?.1 (K), D?.1 (K), D?.1 (K), D?.1 (K), D?.1 (K), D?.1 (K), D?.1 (K), D?.1 (K), D?.1 (K), D?.1 (K)
- new net Row1: D?.1 (K), D?.1 (K), D?.1 (K), D?.1 (K), D?.1 (K), D?.1 (K), D?.1 (K), D?.1 (K), D?.1 (K), D?.1 (K)

Commit message: Finish matrix
Parts:
- added D? (x21): SOD-123, symbol Device:D_Small
- added MX? (x2): Shift, symbol MX_Alps_Hybrid:MX-NoLED
- added MX?: >, symbol MX_Alps_Hybrid:MX-NoLED
- added MX?: <, symbol MX_Alps_Hybrid:MX-NoLED
- added MX?: M, symbol MX_Alps_Hybrid:MX-NoLED
- added MX?: N, symbol MX_Alps_Hybrid:MX-NoLED
- added MX?: B, symbol MX_Alps_Hybrid:MX-NoLED
- added MX?: V, symbol MX_Alps_Hybrid:MX-NoLED
- added MX?: C, symbol MX_Alps_Hybrid:MX-NoLED
- added MX?: X, symbol MX_Alps_Hybrid:MX-NoLED
- added MX?: Z, symbol MX_Alps_Hybrid:MX-NoLED
- added MX?: \\, symbol MX_Alps_Hybrid:MX-NoLED
- added MX?: Ctrl, symbol MX_Alps_Hybrid:MX-NoLED
- added MX?: Win, symbol MX_Alps_Hybrid:MX-NoLED
- added MX?: Alt, symbol MX_Alps_Hybrid:MX-NoLED
- added MX?: Space, symbol MX_Alps_Hybrid:MX-NoLED
- added MX?: Bkspc, symbol MX_Alps_Hybrid:MX-NoLED
- added MX?: Left, symbol MX_Alps_Hybrid:MX-NoLED
- added MX?: Down, symbol MX_Alps_Hybrid:MX-NoLED
- added MX?: Up, symbol MX_Alps_Hybrid:MX-NoLED
- added MX?: Right, symbol MX_Alps_Hybrid:MX-NoLED
Connections:
- net Col0: now also MX?.1 (COL), MX?.1 (COL)
- net Col1: now also MX?.1 (COL), MX?.1 (COL)
- net Col10: now also MX?.1 (COL), MX?.1 (COL)
- net Col11: now also MX?.1 (COL), MX?.1 (COL)
- net Col2: now also MX?.1 (COL), MX?.1 (COL)
- net Col3: now also MX?.1 (COL)
- net Col4: now also MX?.1 (COL)
- net Col5: now also MX?.1 (COL), MX?.1 (COL)
- net Col6: now also MX?.1 (COL)
- net Col7: now also MX?.1 (COL), MX?.1 (COL)
- net Col8: now also MX?.1 (COL), MX?.1 (COL)
- net Col9: now also MX?.1 (COL), MX?.1 (COL)
- new net: D?.2 (A), MX?.2 (ROW) (x21)
- new net Row2: D?.1 (K), D?.1 (K), D?.1 (K), D?.1 (K), D?.1 (K), D?.1 (K), D?.1 (K), D?.1 (K), D?.1 (K), D?.1 (K), D?.1 (K), D?.1 (K)
- new net Row3: D?.1 (K), D?.1 (K), D?.1 (K), D?.1 (K), D?.1 (K), D?.1 (K), D?.1 (K), D?.1 (K), D?.1 (K)

Commit message: assign footprints and make layout
Parts:
- C1, C2, C3, C4, C5, C6: renamed from C?; footprint (none) -> Capacitor_SMD:C_0805_2012Metric
- C7: renamed from C?; footprint (none) -> Diode_SMD:D_SOD-123
- D1, D10, D11, D12, D13, D14, D15, D16, D17, D18, D19, D2, D20, D21, D22, D23, D24, D25, D26, D27, D28, D29, D3, D30, D31, D32, D33, D34, D35, D36, D37, D38, D39, D4, D40, D41, D42, D43, D5, D6, D7, D8, D9: renamed from D?; footprint (none) -> Diode_SMD:D_SOD-123
- MX1, MX41: renamed from MX?; footprint (none) -> MX_Only:MXOnly-ISO-ReversedStabilizers
- MX10, MX12, MX13, MX14, MX15, MX16, MX17, MX18, MX19, MX2, MX20, MX22, MX23, MX24, MX25, MX26, MX27, MX29, MX30, MX31, MX32, MX33, MX34, MX35, MX36, MX37, MX38, MX39, MX4, MX40, MX43, MX5, MX6, MX8, MX9: renamed from MX?; footprint (none) -> MX_Only:MXOnly-1U-NoLED
- MX11, MX3, MX7: renamed from MX?; footprint (none) -> MX_Only:MXOnly-1.25U-NoLED
- MX21: renamed from MX?; footprint (none) -> MX_Only:MXOnly-2.75U-ReversedStabilizers-NoLED
- MX28: renamed from MX?; footprint (none) -> MX_Only:MXOnly-2.25U-ReversedStabilizers-NoLED
- MX42: renamed from MX?; footprint (none) -> MX_Only:MXOnly-1.75U-NoLED
- R1, R2, R4: renamed from R?; footprint (none) -> Resistor_SMD:R_0805_2012Metric
- R3: renamed from R?; value R_Small -> 10k; footprint (none) -> Resistor_SMD:R_0805_2012Metric
- SW1: renamed from SW?; footprint (none) -> random-keyboard-parts:SKQG-1155865
- Y1: renamed from Y?; footprint (none) -> Crystal:Crystal_SMD_3225-4Pin_3.2x2.5mm
- gave numbers to parts that had none: 1

Commit message: place components
Parts:
- C7: footprint Diode_SMD:D_SOD-123 -> Capacitor_SMD:C_0805_2012Metric
Changed lines of the file:
@@
 F 0 "C7" H 2342 2746 50  0000 L CNN
 F 1 "1uF" H 2342 2655 50  0000 L CNN
-F 2 "Diode_SMD:D_SOD-123" H 2250 2700 50  0001 C CNN
+F 2 "Capacitor_SMD:C_0805_2012Metric" H 2250 2700 50  0001 C CNN
 F 3 "~" H 2250 2700 50  0001 C CNN
 	1    2250 2700

Commit message: new layout
Parts:
- MX11, MX3: footprint MX_Only:MXOnly-1.25U-NoLED -> MX_Only:MXOnly-1U-NoLED
- MX2: footprint MX_Only:MXOnly-1U-NoLED -> MX_Only:MXOnly-1.75U-NoLED
- MX31: renamed from MX32; value Left -> /; footprint MX_Only:MXOnly-1U-NoLED -> MX_Only:MXOnly-1.5U-NoLED
- MX36: value Down -> Left
- MX39: renamed from MX6; value \\ -> Up
- MX40: value Up -> Down
- MX42: footprint MX_Only:MXOnly-1.75U-NoLED -> MX_Only:MXOnly-1U-NoLED
- renumbered D14 to D10, D17 to D14, D21 to D15, D15 to D16, D16 to D17, D20 to D18, D18 to D19, D19 to D20, D24 to D21, D27 to D24, D28 to D25, D25 to D26, D26 to D27, D31 to D28, D32 to D31, D35 to D32, D39 to D35, D6 to D39, D10 to D6, MX14 to MX10, MX17 to MX14, MX21 to MX15, MX15 to MX16, MX16 to MX17, MX20 to MX18, MX18 to MX19, MX19 to MX20, MX24 to MX21, MX27 to MX24, MX28 to MX25, MX25 to MX26, MX26 to MX27, MX31 to MX28, MX35 to MX32, MX39 to MX35, MX10 to MX6
Other:
- moved on the sheet: D10, D11, D14, D15, D18, D21, D24, D25, D28, D32, D35, D39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

Commit message: Route matrix and change layout again
Parts:
- MX11: footprint MX_Only:MXOnly-1U-NoLED -> MX_Only:MXOnly-1.25U-NoLED
- MX15: footprint MX_Only:MXOnly-2.75U-ReversedStabilizers-NoLED -> MX_Only:MXOnly-2.25U-ReversedStabilizers-NoLED
- MX25: footprint MX_Only:MXOnly-2.25U-ReversedStabilizers-NoLED -> MX_Only:MXOnly-2U-FLIPPED-ReversedStabilizers
- MX3: footprint MX_Only:MXOnly-1U-NoLED -> MX_Only:MXOnly-1.5U-NoLED
Connections:
- wire segments 176 -> 181
Other:
- moved on the sheet: D15, D31, MX15, MX31
Changed lines of the file:
@@
 F 0 "MX3" H 8233 4455 60  0000 C CNN
 F 1 "Ctrl" H 8233 4365 39  0000 C CNN
-F 2 "MX_Only:MXOnly-1U-NoLED" H 7575 4175 60  0001 C CNN
+F 2 "MX_Only:MXOnly-1.5U-NoLED" H 7575 4175 60  0001 C CNN
 F 3 "" H 7575 4175 60  0001 C CNN
 	1    8200 4200
@@
 F 0 "MX11" H 9533 4455 60  0000 C CNN
 F 1 "Alt" H 9533 4365 39  0000 C CNN
-F 2 "MX_Only:MXOnly-1U-NoLED" H 8875 4175 60  0001 C CNN
+F 2 "MX_Only:MXOnly-1.25U-NoLED" H 8875 4175 60  0001 C CNN
 F 3 "" H 8875 4175 60  0001 C CNN
 	1    9500 4200
@@
 $EndComp
 Wire Wire Line
-	10100 4350 9950 4350
+	10750 4350 10600 4350
 $Comp
 L Device:D_Small D15
 U 1 1 5E11CE36
-P 9950 4450
-F 0 "D15" H 9950 4550 50  0000 R CNN
-F 1 "SOD-123" H 10350 4550 50  0000 R CNN
-F 2 "Diode_SMD:D_SOD-123" V 9950 4450 50  0001 C CNN
-F 3 "~" V 9950 4450 50  0001 C CNN
-	1    9950 4450
+P 10600 4450
+F 0 "D15" H 10600 4550 50  0000 R CNN
+F 1 "SOD-123" H 11000 4550 50  0000 R CNN
+F 2 "Diode_SMD:D_SOD-123" V 10600 4450 50  0001 C CNN
+F 3 "~" V 10600 4450 50  0001 C CNN
+	1    10600 4450
 	0    -1   -1   0
 $EndComp
@@
 L MX_Alps_Hybrid:MX-NoLED MX15
 U 1 1 5E11CE3C
-P 10150 4200
-F 0 "MX15" H 10183 4455 60  0000 C CNN
-F 1 "Space" H 10183 4365 39  0000 C CNN
-F 2 "MX_Only:MXOnly-2.75U-ReversedStabilizers-NoLED" H 9525 4175 60  0001 C CNN
-F 3 "" H 9525 4175 60  0001 C CNN
-	1    10150 4200
+P 10800 4200
+F 0 "MX15" H 10833 4455 60  0000 C CNN
+F 1 "Space" H 10833 4365 39  0000 C CNN
+F 2 "MX_Only:MXOnly-2.25U-ReversedStabilizers-NoLED" H 10175 4175 60  0001 C CNN
+F 3 "" H 10175 4175 60  0001 C CNN
+	1    10800 4200
 	1    0    0    -1
 $EndComp
@@
 F 0 "MX25" H 12083 4455 60  0000 C CNN
 F 1 "Bkspc" H 12083 4365 39  0000 C CNN
-F 2 "MX_Only:MXOnly-2.25U-ReversedStabilizers-NoLED" H 11425 4175 60  0001 C CNN
+F 2 "MX_Only:MXOnly-2U-FLIPPED-ReversedStabilizers" H 11425 4175 60  0001 C CNN
 F 3 "" H 11425 4175 60  0001 C CNN
 	1    12050 4200
@@
 $EndComp
 Wire Wire Line
-	13200 4350 13050 4350
+	13250 4350 13100 4350
 $Comp
 L Device:D_Small D31
 U 1 1 5E14555D
-P 13050 4450
-F 0 "D31" H 13050 4550 50  0000 R CNN
-F 1 "SOD-123" H 13450 4550 50  0000 R CNN
-F 2 "Diode_SMD:D_SOD-123" V 13050 4450 50  0001 C CNN
-F 3 "~" V 13050 4450 50  0001 C CNN
-	1    13050 4450
+P 13100 4450
+F 0 "D31" H 13100 4550 50  0000 R CNN
+F 1 "SOD-123" H 13500 4550 50  0000 R CNN
+F 2 "Diode_SMD:D_SOD-123" V 13100 4450 50  0001 C CNN
+F 3 "~" V 13100 4450 50  0001 C CNN
+	1    13100 4450
 	0    -1   -1   0
 $EndComp
@@
 L MX_Alps_Hybrid:MX-NoLED MX31
 U 1 1 5E145563
-P 13250 4200
-F 0 "MX31" H 13283 4455 60  0000 C CNN
-F 1 "/" H 13283 4365 39  0000 C CNN
-F 2 "MX_Only:MXOnly-1.5U-NoLED" H 12625 4175 60  0001 C CNN
-F 3 "" H 12625 4175 60  0001 C CNN
-	1    13250 4200
+P 13300 4200
+F 0 "MX31" H 13333 4455 60  0000 C CNN
+F 1 "/" H 13333 4365 39  0000 C CNN
+F 2 "MX_Only:MXOnly-1.5U-NoLED" H 12675 4175 60  0001 C CNN
+F 3 "" H 12675 4175 60  0001 C CNN
+	1    13300 4200
 	1    0    0    -1
 $EndComp
@@
 Wire Wire Line
 	8650 4550 8000 4550
-Connection ~ 13050 4550
 Connection ~ 13700 4550
 Wire Wire Line
-	13700 4550 13050 4550
+	13700 4550 13100 4550
 Connection ~ 14300 4550
 Wire Wire Line
@@
 Wire Wire Line
 	8650 4550 9300 4550
-Connection ~ 9950 4550
-Wire Wire Line
-	9950 4550 9300 4550
-Wire Wire Line
-	9950 4550 11850 4550
-Wire Wire Line
-	10300 3300 10300 4150
-Connection ~ 10300 3300
 Connection ~ 11850 4550
 Connection ~ 12200 3300
 Wire Wire Line
-	11850 4550 13050 4550
+	9650 2450 9600 2450
+Connection ~ 9600 2450
+Wire Wire Line
+	10300 2450 10250 2450
+Connection ~ 10250 2450
+Wire Wire Line
+	10950 2450 10900 2450
+Connection ~ 10900 2450
+Wire Wire Line
+	12200 2450 12150 2450
+Connection ~ 12150 2450
+Wire Wire Line
+	13450 2450 13400 2450
+Connection ~ 13400 2450
+Wire Wire Line
+	10950 3300 10950 4150
+Connection ~ 10950 3300
+Connection ~ 10600 4550
+Wire Wire Line
+	10600 4550 11850 4550
+Wire Wire Line
+	9300 4550 10600 4550
+Connection ~ 13100 4550
+Wire Wire Line
+	11850 4550 13100 4550
 $EndSCHEMATC
