File: PeopleMover.kicad_pcb (KiCad board)
At the start: 2 copper layers, 244.5 x 77.8 mm, 106 parts, among them SW1 SW_Push, U1 ATmega32U4-AU, Y1 16MHz

Commit message: Route
Parts:
- moved C5 0.83 mm to (122.1, 74.0)
- moved C2 0.35 mm to (114.5, 57.1)
Routing:
- net Net-(R1-Pad1): track 0.00 -> 174.6 mm, vias 0 -> 4
- net Net-(R2-Pad1): track 0.00 -> 171.1 mm, vias 0 -> 4
- net Net-(R3-Pad2): track 1.89 -> 172.3 mm, vias 0 -> 4
- net GND: track 47.4 -> 168.0 mm, vias 0 -> 4
- net Net-(D38-Pad2): track 0.00 -> 7.31 mm
- net +5V: track 21.6 -> 23.2 mm
